File: Hardware/EnigmaMon.sch (EAGLE design)
At the start: 34 parts, among them T1 BC548, T2 BC548, T3 BC548, T4 BC548, T5 BC548, T6 BC548

Commit message: Added some interesting muxers
Parts:
- removed ARD2: ARD_DIGITAL_1, EnigmaMon:ARD_DIGITAL_1
- removed JP1: (no value), pinhead:PINHD-2X6
- removed JP2: (no value), pinhead:PINHD-1X5
- added C2: 10uF, rcl:C-EU025-025X050
- added D8, D9: 1N4004, diode:1N4004
- added FAN7, FAN8: (no value), pinhead:PINHD-1X3
- added IC1: 4051N, 40xx:4051N
- added IC2: TLC5940, EnigmaMon:TLC5940
- added R15, R17: 1k, rcl:R-EU_0204/7
- added R16, R18, R_BLANK: 10k, rcl:R-EU_0204/7
- added R_IREF: 2.2k, rcl:R-EU_0204/7
- added T8, T9: BC548, transistor:BC547
- added U$1: ARD_POWER, EnigmaMon:ARD_POWER
- added U$2: ARD_DIGITAL_1, EnigmaMon:ARD_DIGITAL_1
- added U$3: ARD_DIGITAL_2, EnigmaMon:ARD_DIGITAL_2
- R1, R4: value (none) -> 10k; device rcl:R-EU_0204/7 -> rcl:R-EU_0207/10
- R10, R12, R6, R8: value (none) -> 10k
- R11, R2, R3, R5, R7, R9: value (none) -> 1k
Connections:
- removed net +5V: JP2.4, R1.2, R10.2, R12.2, R4.2, R6.2, R8.2
- removed net 3.3V: JP2.5
- removed net LCD_DATA: ARD2.3
- new net FAN7_GND: D8.C, FAN7.3, T8.C
- new net FAN7_PWM: IC2G$1.OUT2, R15.1
- new net FAN7_TACHO: FAN7.1, IC1A.X2, R16.1
- new net FAN8_GND: D9.C, FAN8.3, T9.C
- new net FAN8_PWM: IC2G$1.OUT1, R17.1
- new net FAN8_TACHO: FAN8.1, IC1A.X4, R18.1
- new net FAN_TACHO: IC1A.X, U$3.10
- new net N$10: IC2G$1.IREF, R_IREF.1
- new net N$8: R15.2, T8.B
- new net N$9: R17.2, T9.B
- new net PWM_BLANK: IC2G$1.BLANK, R_BLANK.2, U$2.4
- new net PWM_GSCLK: IC2G$1.GSCLK, U$2.5
- new net PWM_SCLK: IC2G$1.SCLK, U$2.7
- new net PWM_SIN: IC2G$1.SIN, U$3.8
- new net PWM_VPRG: IC2G$1.VPRG, U$3.9
- new net PWM_XLAT: IC2G$1.XLAT, U$2.6
- new net TACHO_SEL0: IC1A.A, U$3.11
- new net TACHO_SEL1: IC1A.B, U$3.12
- new net TACHO_SEL2: IC1A.C, U$3.13
- new net VCC: C2.1, IC2G$1.DCPRG, R1.2, R10.2, R12.2, R16.2, R18.2, R4.2, R6.2, R8.2, R_BLANK.1, U$1.5V
- net +12V: now also FAN7.2, FAN8.2, U$1.VIN; no longer JP2.1
- net FAN1_PWM: now also IC2G$1.OUT8; no longer JP1.2
- net FAN1_TACHO: now also IC1A.X3; no longer JP1.1
- net FAN2_PWM: now also IC2G$1.OUT7; no longer JP1.4
- net FAN2_TACHO: now also IC1A.X5; no longer JP1.3
- net FAN3_PWM: now also IC2G$1.OUT6; no longer JP1.6
- net FAN3_TACHO: now also IC1A.X0; no longer JP1.5
- net FAN4_PWM: now also IC2G$1.OUT5; no longer JP1.8
- net FAN4_TACHO: now also IC1A.X7; no longer JP1.7
- net FAN5_PWM: now also IC2G$1.OUT4; no longer JP1.10
- net FAN5_TACHO: now also IC1A.X1; no longer JP1.9
- net FAN6_PWM: now also IC2G$1.OUT3; no longer JP1.12
- net FAN6_TACHO: now also IC1A.X6; no longer JP1.11
- net GND: now also C2.2, D8.A, D9.A, IC1A.INH, R_IREF.2, T8.E, T9.E, U$1.GND@1, U$1.GND@2, U$3.GND; no longer JP2.2, JP2.3
Other:
- moved on the sheet: D1, D2, D3, D4, D5, D6, FAN1, FAN2, FAN3, FAN4, FAN5, FAN6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

Commit message: Added some interesting muxers
Parts:
- PWR: value PIN02-1V -> (none); device EnigmaMon:PIN02-1V -> EnigmaMon:PINHD-1X2
Other:
- moved on the sheet: PWR, U$2, U$3
